File: eagle/Design/Pi.brd (EAGLE design)
At the start: 66.2 x 57.3 mm, 26 parts, among them IC1 LM340S, IC2 DS2484, IC3 PAM8403, Q1 SI2369DS, SW1 SWITCH, X1 SUPPLY_12V, X3 PG203J

Commit message: Completed schematic and board routing for Pi controller.
Assuming I don't find any last minute issues this will be the final
revision of version 1.0.
Parts:
- removed LED1, LED2: (no value), led:CHIP-LED0805
- added C9: 1u, resistor:C0603
- added LED-G: (no value), led:CHIP-LED0603
- added Q2: SI2342DS, Custom:SOT23
- C5: value 470u -> 100u; device resistor:C0603 -> rcl:C0805
- moved R2 34.0 mm to (6.22, 20.1), turned to 180 degrees
- moved R1 23.2 mm to (51.8, 43.8), turned to 0 degrees
- moved IC2 21.3 mm to (29.6, 37.3)
- moved C5 4.95 mm to (22.1, 26.5)
- moved F1 4.54 mm to (52.9, 22.2), flipped to the bottom, turned to 90 degrees
- moved C1 0.64 mm to (22.2, 43.8)
- moved C2 0.64 mm to (17.7, 43.8)
Connections:
- removed net LED_GREEN: LED2.C, PCB1.19
- removed net LED_RED: LED1.C, PCB1.21
- removed net N$7: IC2.5, X2.6
- new net !1WIRE_SLP: IC2.1, PCB1.7
- new net !AMP_MUTE: IC3.5, PCB1.23
- new net !AMP_SHDN: IC3.12, PCB1.21
- new net !LED_GREEN: PCB1.33, Q2.1
- new net N$20: LED-G.C, Q2.3
- new net OW: IC2.5, X2.7
- net +12V: now also X2.3, X2.4; no longer X2.1, X2.2
- net +3P3V: now also X2.8; no longer R2.2, X2.5
- net +5V: now also C9.1, X2.5, X2.6; no longer X2.3, X2.4
- net GND: now also C9.2, Q2.2, R2.1, X2.1, X2.2; no longer SW1.3, X2.7, X2.8
- net N$1: now also LED-G.A; no longer LED1.A
- net N$2: now also R2.2, SW1.3; no longer LED2.A, R2.1
Routing:
- net +3P3V: track 10.4 -> 70.3 mm
- net !AMP_SHDN: track 0.00 -> 36.5 mm, vias 0 -> 2
- net +5V: track 92.4 -> 128.8 mm
- net OW: track 0.00 -> 33.2 mm
- net !AMP_MUTE: track 0.00 -> 30.1 mm, vias 0 -> 2
- net !1WIRE_SLP: track 0.00 -> 25.2 mm
- net N$6: track 50.0 -> 26.4 mm, vias 1 -> 0
- net N$5: track 54.2 -> 31.9 mm, vias 1 -> 0
- net LED_RED: track 22.2 -> 0.00 mm
- net LED_GREEN: track 15.6 -> 0.00 mm
- net N$7: track 9.97 -> 0.00 mm
- net !LED_GREEN: track 0.00 -> 7.48 mm
- net N$20: track 0.00 -> 6.91 mm
- net N$13: track 79.4 -> 85.9 mm, vias 3 -> 0
- net +12V: track 16.6 -> 12.9 mm
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Other:
- outline, holes or cut-outs redrawn
- board text added: "+"
- board text added: "-"
- board text added: "Uber Brew"
- board text added: "v1.0"
