File: eagle/Design/Pi.sch (EAGLE design)
At the start: 28 parts, among them IC1 LM340S, IC2 DS2484, IC3 PAM8403, Q1 SI2369DS, SW1 SWITCH, X1 SUPPLY_12V, X3 PG203J

Commit message: Completed schematic and board routing for Pi controller.
Assuming I don't find any last minute issues this will be the final
revision of version 1.0.
Parts:
- removed LED1, LED2: (no value), led:LEDCHIP-LED0805
- added C9: 1u, resistor:C-USC0603
- added LED-G: (no value), led:LEDCHIP-LED0603
- added Q2: SI2342DS, Custom:SI2342DS
- C5: value 470u -> 100u; device resistor:C-USC0603 -> rcl:C-USC0805
Connections:
- removed net LED_GREEN: LED2.C, PCB1-GPIO.GPIO10
- removed net LED_RED: LED1.C, PCB1-GPIO.GPIO9
- removed net N$7: IC2.IO, X2.P$6
- new net !1WIRE_SLP: IC2.!SLP, PCB1-GPIO.GPIO4
- new net !AMP_MUTE: IC3.!MUTE, PCB1-GPIO.GPIO11
- new net !AMP_SHDN: IC3.!SHDN, PCB1-GPIO.GPIO9
- new net !LED_GREEN: PCB1-GPIO.GPIO13, Q2.G
- new net N$20: LED-G.C, Q2.D
- new net OW: IC2.IO, X2.P$7
- net +12V: now also X2.P$3, X2.P$4; no longer X2.P$1, X2.P$2
- net +3P3V: now also X2.P$8; no longer R2.2, X2.P$5
- net +5V: now also C9.1, X2.P$5, X2.P$6; no longer X2.P$3, X2.P$4
- net GND: now also C9.2, Q2.S, R2.1, X2.P$1, X2.P$2; no longer SW1.S, X2.P$7, X2.P$8
- net N$1: now also LED-G.A; no longer LED1.A
- net N$2: now also R2.2, SW1.S; no longer LED2.A, R2.1
Other:
- moved on the sheet: R1, R2, X2
